Commit message: Updated parameters and launch file

File: jetsoncar_description/urdf/jetsoncar.xacro (robot description, xacro)
@@ -11,8 +11,8 @@
      and https://github.com/mit-racecar/racecar-simulator/blob/master/racecar_description/urdf/racecar.xacro
 -->
-	<xacro:include filename="$(find jetsoncar_sim_description)/urdf/parameters.xacro" />
-	<xacro:include filename="$(find jetsoncar_sim_description)/urdf/physical.xacro" />
-	<xacro:include filename="$(find jetsoncar_sim_description)/urdf/joints.xacro" />
-	<xacro:include filename="$(find jetsoncar_sim_description)/urdf/materials.xacro" />
+	<xacro:include filename="$(find jetsoncar_description)/urdf/parameters.xacro" />
+	<xacro:include filename="$(find jetsoncar_description)/urdf/physical.xacro" />
+	<xacro:include filename="$(find jetsoncar_description)/urdf/joints.xacro" />
+	<xacro:include filename="$(find jetsoncar_description)/urdf/materials.xacro" />
 	<link name="footprint"/>
 	<link name="base_link">

File: jetsoncar_description/urdf/joints.xacro (robot description, xacro)
@@ -1,5 +1,5 @@
 <?xml version="1.0"?>
 <robot name="jetsoncar" xmlns:xacro="http://www.ros.org/wiki/xacro">
-	<xacro:include filename="$(find jetsoncar_sim_description)/urdf/parameters.xacro" />
+	<xacro:include filename="$(find jetsoncar_description)/urdf/parameters.xacro" />
 	<xacro:macro name="fixed_offset_joint" params="parent child offset">
 		<joint name="${parent}_to_${child}" type="fixed">

File: jetsoncar_description/urdf/parameters.xacro (robot description, xacro)
@@ -2,11 +2,11 @@
 <robot name="jetsoncar" xmlns:xacro="http://www.ros.org/wiki/xacro">
 	<!-- X axis direction is forward, Y axis direction is left -->
-    <!-- Sensors related properties -->
-    <xacro:property name="enable_lidar" value="true" />
-    <xacro:property name="enable_realsense" value="false" />
-    <xacro:property name="enable_range_sensors" value="false" />
-    <xacro:property name="enable_dual_camera" value="true" />
-    <xacro:property name="enable_front_camera" value="false" />
-    <xacro:property name="enable_imu" value="true" />
+	<!-- Sensors related properties -->
+	<xacro:property name="enable_lidar" value="true" />
+	<xacro:property name="enable_realsense" value="false" />
+	<xacro:property name="enable_range_sensors" value="false" />
+	<xacro:property name="enable_dual_camera" value="true" />
+	<xacro:property name="enable_front_camera" value="false" />
+	<xacro:property name="enable_imu" value="true" />
 	<!-- IMU related properties -->
 	<xacro:property name="imu_width" value="0.05" />
@@ -57,3 +57,5 @@
 	<xacro:property name="ranger_height" value="0.02" />
 	<xacro:property name="ranger_weight" value="0.050" />
+	<!-- Steering related properties -->
+	<xacro:property name="steering_wheel_angle_limit" value="${40/180*pi}" />
 </robot>

File: jetsoncar_description/urdf/physical.xacro (robot description, xacro)
@@ -2,5 +2,5 @@
 <robot name="jetsoncar" xmlns:xacro="http://www.ros.org/wiki/xacro">
 	<!-- X axis direction is forward, Y axis direction is left -->
-	<xacro:include filename="$(find jetsoncar_sim_description)/urdf/parameters.xacro" />
+	<xacro:include filename="$(find jetsoncar_description)/urdf/parameters.xacro" />
 	<!-- IMU -->
 	<xacro:macro name="imu_geometry">
